File: PCB/Doorlockd-Controller.kicad_pcb (KiCad board)
At the start: 2 copper layers, 132 x 103 mm, 60 parts, among them J1 MilkV P43 (3.3V for VCCB), J10 Power Out 1, J11 DC in, J12 IO 3, J13 Debug UART, J14 IO 4, J15 Power Out 2, J16 to extra screw conn., J18 GPIO only MilkV 1.8V, J19 3V 5V Vin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

Commit message: Change LED resistors to 220
This reduces LED current a bit, and reduces BOM count.
Parts:
- R1, R4: value 100 -> 220
Changed lines of the file:
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@@
 			)
 		)
-		(property "Value" "100"
+		(property "Value" "220"
 			(at 5.08 2.37 0)
 			(layer "F.Fab")
@@
 			)
 		)
-		(property "Value" "100"
+		(property "Value" "220"
 			(at 5.08 2.37 0)
 			(layer "F.Fab")

Commit message: Some silkscreen tweaks
Other:
- board text added: "+"
- board text added: "-"
- board text added: "CPU Board Rock Pi S or Milk-V Duo S"
- board text added: "feed 5V to CPU board"
- board text added: "select Out5 +"
- board text added: "select Out6 +"
- board text removed: "backfeed 5V to PC"
- board text removed: "select V Out 5"
- board text removed: "select V Out 6"

Commit message: Use correct IPAK footprint
This used the SIPAK footprint, but that is slightly different (and has
no 3D model), so use the IPAK/TO-251-3 footprint instead.
Parts:
- Q2, Q5: footprint Package_TO_SOT_THT:SIPAK_Vertical -> Package_TO_SOT_THT:TO-251-3_Vertical
