File: PCB/Doorlockd-Controller.kicad_sch (KiCad schematic)
At the start: 59 parts, among them J1 MilkV P43 (3.3V for VCCB), J10 Power Out 1, J11 DC in, J12 IO 3, J13 Debug UART, J14 IO 4, J15 Power Out 2, J16 to extra screw conn., J18 GPIO only MilkV 1.8V, J19 3V 5V Vin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

Commit message: made title, boardname and silk consistent
Other:
- title: Doorlockd Controller PCB -> Doorlockd PCB Controller
Changed lines of the file:
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@@
 	(paper "A4")
 	(title_block
-		(title "Doorlockd Controller PCB")
+		(title "Doorlockd PCB Controller")
 		(date "2025-06-17")
 		(comment 1 "Copyright 2025 Diederik Hamelink (wie-niet) & Matthijs Kooijman")
